File: Schematics_&_PCB/inverted_pendulum_shield/inverted_pendulum_shield.kicad_pcb (KiCad board)
At the start: 2 copper layers, 77 x 73 mm, 52 parts, among them J1 Screw_Terminal_01x02, J2 Screw_Terminal_01x04, J3 Screw_Terminal_01x02, J4 FCR7350R, J5 FCR7350B, Q1 DMP3056L-7, Q2 NX138BKR, Q3 FQD8P10TM, Q4 SLMT320V3CN, Q5 SLMT320V3CN, SW1 1825027, U1 DRV8231DDAR, U2 AP63301WU-7

Commit message: fixed a couple comment errors
Other:
- board text added: "RPP"
- board text removed: "RVP"
