File: Schematics_&_PCB/inverted_pendulum_shield/inverted_pendulum_shield.kicad_sch (KiCad schematic)
At the start: 52 parts, among them J1 Screw_Terminal_01x02, J2 Screw_Terminal_01x04, J3 Screw_Terminal_01x02, J4 FCR7350R, J5 FCR7350B, Q1 DMP3056L-7, Q2 NX138BKR, Q3 FQD8P10TM, Q4 SLMT320V3CN, Q5 SLMT320V3CN, SW1 1825027, U1 DRV8231DDAR, U2 AP63301WU-7

Commit message: changed readme layout
Other:
- note added: "Supply with RPP & Voltage reading"
- note removed: "Supply with RVP & Voltage reading"
Changed lines of the file:
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@@
 		)
 	)
-	(text "Supply with RVP & Voltage reading"
+	(text "Supply with RPP & Voltage reading"
 		(exclude_from_sim no)
 		(at 53.848 138.938 0)

Commit message: fixed a couple comment errors
Other:
- note added: "5/180 = 27.8mA"
- note removed: "5/330 = 15mA"
Changed lines of the file:
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@@
 		)
 	)
-	(text "5/330 = 15mA"
+	(text "5/180 = 27.8mA"
 		(exclude_from_sim no)
-		(at 309.372 209.804 0)
+		(at 310.134 209.804 0)
 		(effects
 			(font
@@
 	(text "Raspberry Pi Pico connections"
 		(exclude_from_sim no)
-		(at 187.96 81.28 0)
+		(at 175.514 81.534 0)
 		(effects
 			(font
